File: placa/ESP32-DevKitC/esp32-devkitc_template.kicad_pcb (KiCad board)
At the start: 2 copper layers, 50 x 80 mm, 1 part, among them U1 ESP32-DevKitC

Commit message: m
Parts:
- added C12V1: 10uF, Capacitor_THT:CP_Radial_Tantal_D5.5mm_P2.50mm, F.Cu at (157.5, 67.5)
- added C3.3V1: 10uF, Capacitor_THT:CP_Radial_Tantal_D5.5mm_P2.50mm, F.Cu at (158.5, 56.2)
- added C5V1: 10uF, Capacitor_THT:CP_Radial_Tantal_D5.5mm_P2.50mm, F.Cu at (158.0, 60.5)
- added Cf1: 10nF, Capacitor_THT:C_Rect_L4.6mm_W2.0mm_P2.50mm_MKS02_FKP02, F.Cu at (164.0, 56.3)
- added Cf2: 10nF, Capacitor_THT:C_Rect_L4.6mm_W2.0mm_P2.50mm_MKS02_FKP02, F.Cu at (163.0, 61.0)
- added Cf3: 10nF, Capacitor_THT:C_Rect_L4.6mm_W2.0mm_P2.50mm_MKS02_FKP02, F.Cu at (163.0, 67.7)
- added JCOOLER1: Conn_01x03, Connector_PinHeader_2.54mm:PinHeader_1x03_P2.54mm_Vertical, F.Cu at (144.5, 53.5)
- added JDISPLAY1: Conn_01x04, Connector_PinSocket_2.54mm:PinSocket_1x04_P2.54mm_Vertical, F.Cu at (158.0, 40.0)
- added JENCODER1: Conn_01x05, Connector_PinSocket_2.54mm:PinSocket_1x05_P2.54mm_Vertical, F.Cu at (144.5, 57.3)
- added JFUENTE1: Conn_01x04, TerminalBlock:TerminalBlock_Xinya_XY308-2.54-4P_1x04_P2.54mm_Horizontal, F.Cu at (171.5, 60.3)
- added JIN1: Conn_01x02, Connector_PinHeader_2.54mm:PinHeader_1x02_P2.54mm_Vertical, F.Cu at (145.5, 23.5)
- added JSD1: Conn_01x06, Connector_PinHeader_2.54mm:PinHeader_1x06_P2.54mm_Vertical, F.Cu at (165.5, 46.6)
- U1: footprint Espressif:ESP32-DevKitC -> PCM_Espressif:ESP32-DevKitC
- moved U1 45.8 mm to (110.3, 27.6)
Connections:
- U1 pad 1: unconnected-(U1-Pad1) -> +3V3
- U1 pad 10: unconnected-(U1-Pad10) -> /GPIO26
- U1 pad 11: unconnected-(U1-Pad11) -> /GPIO27
- U1 pad 12: unconnected-(U1-Pad12) -> /GPIO14
- U1 pad 13: unconnected-(U1-Pad13) -> /GPIO12
- U1 pad 15: unconnected-(U1-Pad15) -> /GPIO13
- U1 pad 16: unconnected-(U1-Pad16) -> /SD2
- U1 pad 17: unconnected-(U1-Pad17) -> /SD3
- U1 pad 18: unconnected-(U1-Pad18) -> /CMD
- U1 pad 20: unconnected-(U1-Pad20) -> /SDCLK
- U1 pad 21: unconnected-(U1-Pad21) -> /SD0
- U1 pad 22: unconnected-(U1-Pad22) -> /SD1
- U1 pad 23: unconnected-(U1-Pad23) -> /GPIO15
- U1 pad 24: unconnected-(U1-Pad24) -> /SW
- U1 pad 25: unconnected-(U1-Pad25) -> /OUTA
- U1 pad 26: unconnected-(U1-Pad26) -> /OUTB
- U1 pad 27: unconnected-(U1-Pad27) -> /COOLER
- U1 pad 28: unconnected-(U1-Pad28) -> /GPIO17
- U1 pad 29: unconnected-(U1-Pad29) -> /CS
- U1 pad 3: unconnected-(U1-Pad3) -> /SVP I/O
- U1 pad 30: unconnected-(U1-Pad30) -> /SCK
- U1 pad 31: unconnected-(U1-Pad31) -> /MISO
- U1 pad 33: unconnected-(U1-Pad33) -> /SDA
- U1 pad 34: unconnected-(U1-Pad34) -> /RX
- U1 pad 35: unconnected-(U1-Pad35) -> /TX
- U1 pad 36: unconnected-(U1-Pad36) -> /SCL
- U1 pad 37: unconnected-(U1-Pad37) -> /MOSI
- U1 pad 4: unconnected-(U1-Pad4) -> /SVN I/O
- U1 pad 5: unconnected-(U1-Pad5) -> /GPIO34 I/O
- U1 pad 6: unconnected-(U1-Pad6) -> /GPIO35 I/O
- U1 pad 7: unconnected-(U1-Pad7) -> /GPIO32
- U1 pad 8: unconnected-(U1-Pad8) -> /GPIO33
- U1 pad 9: unconnected-(U1-Pad9) -> /GPIO25
Routing:
- net +3V3: track 0.00 -> 174.4 mm
- net +5V: track 0.00 -> 108.0 mm, vias 0 -> 2
- net /MOSI: track 0.00 -> 46.6 mm
- net +12V: track 0.00 -> 44.0 mm, vias 0 -> 2
- net /CS: track 0.00 -> 38.0 mm, vias 0 -> 2
- net /MISO: track 0.00 -> 36.8 mm
- net /SCK: track 0.00 -> 33.5 mm
- net /RX: track 0.00 -> 30.9 mm
- net /SCL: track 0.00 -> 24.3 mm
- net /SDA: track 0.00 -> 22.4 mm
- net /TX: track 0.00 -> 21.9 mm
- net /COOLER: track 0.00 -> 10.7 mm
- net /OUTB: track 0.00 -> 9.11 mm
- net /OUTA: track 0.00 -> 9.11 mm
- net /SW: track 0.00 -> 9.11 mm
- added copper zone on B.Cu, net GND
Other:
- board outline removed
