File: placa/ESP32-DevKitC/esp32-devkitc_template.kicad_sch (KiCad schematic)
At the start: 18 parts, among them U1 ESP32-DevKitC

Commit message: m
Parts:
- removed A? (x3): Pololu_Breakout_A4988, Module:Pololu_Breakout-16_15.2x20.3mm, symbol Driver_Motor:Pololu_Breakout_A4988
- removed CMOT0, CMOT1, CMOT2: C, symbol Device:C
- removed JMOT0, JMOT1, JMOT2: Conn_01x04_Pin, symbol Connector:Conn_01x04_Pin
- removed JMOT0LS, JMOT0MS, JMOT1LS, JMOT1MS, JMOT2LS, JMOT2MS: Conn_01x03_Pin, symbol Connector:Conn_01x03_Pin
- removed JPOWER: Conn_01x06, symbol Connector_Generic:Conn_01x06
- removed JTARJETASD: Conn_01x08_Pin, symbol Connector:Conn_01x08_Pin
- added C12V1, C3.3V1, C5V1: 10uF, Capacitor_THT:CP_Radial_Tantal_D5.5mm_P2.50mm, symbol Device:C
- added Cf1, Cf2, Cf3: 10nF, Capacitor_THT:C_Rect_L4.6mm_W2.0mm_P2.50mm_MKS02_FKP02, symbol Device:C
- added JCOOLER1: Conn_01x03, Connector_PinHeader_2.54mm:PinHeader_1x03_P2.54mm_Vertical, symbol Connector_Generic:Conn_01x03
- added JDISPLAY1: Conn_01x04, Connector_PinSocket_2.54mm:PinSocket_1x04_P2.54mm_Vertical, symbol Connector_Generic:Conn_01x04
- added JENCODER1: Conn_01x05, Connector_PinSocket_2.54mm:PinSocket_1x05_P2.54mm_Vertical, symbol Connector_Generic:Conn_01x05
- added JFUENTE1: Conn_01x04, Connector_PinHeader_2.54mm:PinHeader_1x04_P2.54mm_Vertical, symbol Connector_Generic:Conn_01x04
- added JIN1: Conn_01x02, Connector_PinHeader_2.54mm:PinHeader_1x02_P2.54mm_Vertical, symbol Connector_Generic:Conn_01x02
- added JSD1: Conn_01x06, Connector_PinHeader_2.54mm:PinHeader_1x06_P2.54mm_Vertical, symbol Connector_Generic:Conn_01x06
- U1: footprint Espressif:ESP32-DevKitC -> PCM_Espressif:ESP32-DevKitC
Connections:
- net +12V: now also C12V1.1, Cf3.1, JCOOLER1.3 (Pin_3), JFUENTE1.2 (Pin_2)
- net +3V3: now also C3.3V1.1, Cf1.1, JFUENTE1.3 (Pin_3), JSD1.3 (Pin_3)
- net +5V: now also C5V1.1, Cf2.1, JDISPLAY1.3 (Pin_3), JENCODER1.4 (Pin_4), JFUENTE1.1 (Pin_1)
- net CS: now also JSD1.1 (Pin_1)
- net GND: now also C12V1.2, C3.3V1.2, C5V1.2, Cf1.2, Cf2.2, Cf3.2, JCOOLER1.1 (Pin_1), JDISPLAY1.4 (Pin_4), JENCODER1.5 (Pin_5), JFUENTE1.4 (Pin_4), JSD1.5 (Pin_5)
- net MISO: now also JSD1.6 (Pin_6)
- net MOSI: now also JSD1.2 (Pin_2)
- net RX: now also JIN1.1 (Pin_1)
- net SCK: now also JSD1.4 (Pin_4)
- net TX: now also JIN1.2 (Pin_2)
- net GPIO0 renamed OUTA
- net OUTA: now also JENCODER1.2 (Pin_2)
- net GPIO16 renamed COOLER
- net COOLER: now also JCOOLER1.2 (Pin_2)
- net GPIO2 renamed SW
- net SW: now also JENCODER1.3 (Pin_3)
- net GPIO21 renamed SDA
- net SDA: now also JDISPLAY1.1 (Pin_1)
- net GPIO22 renamed SCL
- net SCL: now also JDISPLAY1.2 (Pin_2)
- net GPIO4 renamed OUTB
- net OUTB: now also JENCODER1.1 (Pin_1)
Other:
- note added: "COOLER"
- note added: "DISPLAY"
- note added: "ENCODER"
- note added: "ENTRADA"
- note added: "FILTROS CAPACITIVOS"
- note removed: "FIN DE CARRERA"
